File: splave-ferris_choc_v1/output/pcbs/splave-ferris_choc_v1_left.kicad_pcb (KiCad board)
At the start: 2 copper layers, 130.2 x 101.2 mm, 38 parts

Commit message: Finalized choc_v1 design and created production files.
Parts:
- moved D1 279.5 mm to (120.0, 215.0)
- moved D2 279.5 mm to (120.0, 198.0)
- moved D3 279.5 mm to (120.0, 181.0)
- moved S1 279.5 mm to (120.0, 210.0)
- moved S2 279.5 mm to (120.0, 193.0)
- moved S3 279.5 mm to (120.0, 176.0)
- moved D4 240.6 mm to (139.5, 203.0), turned to -6 degrees
- moved S4 239.5 mm to (140.0, 198.0), turned to -6 degrees
- moved D5 237.0 mm to (141.3, 186.1), turned to -6 degrees
- moved S5 236.0 mm to (141.8, 181.1), turned to -6 degrees
- moved D6 233.5 mm to (143.0, 169.2), turned to -6 degrees
- moved S6 232.4 mm to (143.6, 164.2), turned to -6 degrees
- moved D7 201.9 mm to (158.8, 198.0), turned to -9 degrees
- moved S7 200.3 mm to (159.6, 193.0), turned to -9 degrees
- moved D8 196.5 mm to (161.5, 181.2), turned to -9 degrees
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Connections:
- net mirror_far_fan renamed far_fan
- net mirror_index_bottom renamed index_bottom
- net mirror_index_home renamed index_home
- net mirror_index_top renamed index_top
- net mirror_inner_bottom renamed inner_bottom
- net mirror_inner_home renamed inner_home
- net mirror_inner_top renamed inner_top
- net mirror_middle_bottom renamed middle_bottom
- net mirror_middle_home renamed middle_home
- net mirror_middle_top renamed middle_top
- net mirror_near_fan renamed near_fan
- net mirror_pinky_bottom renamed pinky_bottom
- net mirror_pinky_home renamed pinky_home
- net mirror_pinky_top renamed pinky_top
- net mirror_ring_bottom renamed ring_bottom
- net mirror_ring_home renamed ring_home
- net mirror_ring_top renamed ring_top
- B1 pad 1: RST -> GND
- B1 pad 2: GND -> RST
- D1 pad 1: D2 -> D5
- D10 pad 1: D2 -> D5
- D11 pad 1: D1 -> D3
- D13 pad 1: D2 -> D5
- D14 pad 1: D1 -> D3
- D16 pad 1: D4 -> D9
- D17 pad 1: D4 -> D9
- D2 pad 1: D1 -> D3
- D4 pad 1: D2 -> D5
- D5 pad 1: D1 -> D3
- D7 pad 1: D2 -> D5
- D8 pad 1: D1 -> D3
- S1 pad 2: D8 -> D4
- S10 pad 2: D3 -> D10
- S11 pad 2: D3 -> D10
- S12 pad 2: D3 -> D10
- S13 pad 2: D5 -> D8
- S14 pad 2: D5 -> D8
- S15 pad 2: D5 -> D8
- S16 pad 2: D3 -> D10
- S17 pad 2: D5 -> D8
- S2 pad 2: D8 -> D4
- S3 pad 2: D8 -> D4
- S4 pad 2: D10 -> D2
- S5 pad 2: D10 -> D2
- S6 pad 2: D10 -> D2
- S7 pad 2: D9 -> D1
- S8 pad 2: D9 -> D1
- S9 pad 2: D9 -> D1
- T1 pad 1: BAT -> BATCON
- T1 pad 2: BATCON -> BAT
Other:
- outline, holes or cut-outs redrawn
