File: splave-ferris_pg1316s/splave-ferris_pg1316s_unrouted.kicad_pcb (KiCad board)
At the start: 2 copper layers, 242.9 x 85.9 mm, 74 parts

Commit message: Add stablizer holes to PG1316S footprint, regenerate PCB files.
Parts:
- S1, S10, S11, S12, S13, S14, S15, S16, S17, S18, S19, S2, S20, S21, S22, S23, S24, S25, S26, S27, S28, S29, S3, S30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: footprint PG1316S -> CPG1316S01D02_mikeholscher
Other:
- net class Default added: clearance 0.2, trace_width 0.25, via_dia 0.8, via_drill 0.4
